File: Hardware/gator-bit.brd (EAGLE design)
At the start: 114.4 x 70.4 mm, 93 parts, among them J1 GATOR, J10 GATOR, J11 GATOR, J12 GATOR, J13 GATOR, J14 GATOR, J15 GATOR, J16 GATOR, J17 GATOR, J18 GATOR, J2 GATOR, J3 GATOR, J4 GATOR, J6 GATOR, J7 GATOR, J8 GATOR, J9 GATOR, U1 TPS63070, U2 micro:bit, U3 TXB0104, U4 ADJ REG 1.5A

Commit message: v02, silk
Parts:
- moved LOGO6 105.6 mm to (109.3, 4.22)
- moved R23 15.5 mm to (96.9, 45.8), turned to 270 degrees
- moved R22 14.3 mm to (97.8, 62.8), turned to 270 degrees
- moved FD3 11.7 mm to (109.2, 4.20)
- moved D9 7.67 mm to (97.7, 56.7), turned to 90 degrees
- moved D11 7.45 mm to (97.6, 38.9), turned to 90 degrees
- moved LOGO5 4.60 mm to (26.7, 33.6)
- moved U3 3.58 mm to (26.9, 28.5)
- moved R19 1.15 mm to (77.6, 16.6)
- moved D19 1.15 mm to (77.3, 20.8)
- moved R20 1.15 mm to (77.6, 18.5)
- moved R9 1.10 mm to (87.5, 16.7)
- moved D10 1.10 mm to (87.2, 20.8)
- moved R10 1.10 mm to (87.5, 18.6)
- moved R17 1.09 mm to (47.0, 16.7)
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Routing:
- net GND: track 79.5 -> 68.7 mm
- net P12LL: track 28.7 -> 34.6 mm
- net VSUPPLY: track 42.0 -> 46.3 mm
- net P12: track 6.01 -> 9.68 mm
- net N$24: track 2.08 -> 5.47 mm
- net P5+: track 15.5 -> 12.2 mm
- net 3.3V: track 140.6 -> 143.6 mm
- net N$23: track 1.77 -> 4.46 mm
- net P5: track 55.0 -> 57.5 mm
- net VOUT5.0: track 22.5 -> 24.5 mm
- net P16: track 27.3 -> 28.9 mm
- net P2: track 39.6 -> 40.9 mm
- net 5V: track 138.6 -> 139.8 mm
- net P2+: track 16.2 -> 15.1 mm
- net P8+: track 15.6 -> 14.5 mm
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Other:
- board text added: "v02"
- board text removed: "v01"
