File: Hardware/Production/gator-bit-Panel.brd (EAGLE design)
At the start: 357.8 x 155 mm, 537 parts, among them J1 GATOR, J10 GATOR, J100 GATOR, J101 GATOR, J102 GATOR, J103 GATOR, J104 GATOR, J105 GATOR, J106 GATOR, J107 GATOR, J11 GATOR, J12 GATOR, J13 GATOR, J14 GATOR, J15 GATOR, J16 GATOR, J17 GATOR, J18 GATOR, J19 GATOR, J2 GATOR, J20 GATOR, J21 GATOR, J22 GATOR, J23 GATOR, J24 GATOR, J25 GATOR, J26 GATOR, J27 GATOR, J28 GATOR, J29 GATOR, J3 GATOR, J30 GATOR, J31 GATOR, J32 GATOR, J33 GATOR, J34 GATOR, J35 GATOR, J37 GATOR, J38 GATOR, J39 GATOR, J4 GATOR, J40 GATOR, J41 GATOR, J42 GATOR, J43 GATOR, J44 GATOR, J45 GATOR, J46 GATOR, J47 GATOR, J48 GATOR, J49 GATOR, J50 GATOR, J51 GATOR, J52 GATOR, J53 GATOR, J55 GATOR, J56 GATOR, J57 GATOR, J58 GATOR, J59 GATOR, J6 GATOR, J60 GATOR, J61 GATOR, J62 GATOR, J63 GATOR, J64 GATOR, J65 GATOR, J66 GATOR, J67 GATOR, J68 GATOR, J69 GATOR, J7 GATOR, J70 GATOR, J71 GATOR, J73 GATOR, J74 GATOR, J75 GATOR, J76 GATOR, J77 GATOR, J78 GATOR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

Commit message: panel
Parts:
- removed F1, F2, F3, F4, F5, F6: 6V/0.5A, SparkFun-Fuses:1206
- removed R109, R132: 523k, SparkFun-Resistors:0603
- removed R110, R130, R133: 100k, SparkFun-Resistors:0603
- removed R111, R134: 390k, SparkFun-Resistors:0603
- removed R112, R135: 240, SparkFun-Resistors:0603
- removed R113, R114, R115, R136, R137, R138: 1k, SparkFun-Resistors:0603
- removed R116, R118, R120, R122, R124, R126, R128: 604, SparkFun-Resistors:0603
- removed R117, R119, R121, R123, R125, R127, R129: 910, SparkFun-Resistors:0603
- removed R131: 10.2K, SparkFun-Resistors:0603
- removed S13, S14, S15, S16, S17, S18, S19, S20, S21, S22, S23, S24: (no value), SparkFun-Switches:SWITCH_DPDT_SMD_AYZ0202
- added D100, D97, D98, D99: WS2812B, SparkFun-LED:WS2812B
- added D101, D102, D103, D104, D105, D106, D107: 3.6V, SparkFun-DiscreteSemi:SOD-323
- added D108, D112, D113: 1A/23V/620mV, SparkFun-DiscreteSemi:SOD-323
- added D109, D110, D111: RED, SparkFun-LED:LED-0603
- added D114: 120mA/40V/370mV, SparkFun-DiscreteSemi:SOD-523
- added FRAME1, FRAME10, FRAME11, FRAME12, FRAME2, FRAME3, FRAME4, FRAME5, FRAME6, FRAME7, FRAME8, FRAME9: FRAME-LETTER, SparkFun-Aesthetics:CREATIVE_COMMONS
- added H1, H10, H11, H12, H2, H3, H4, H5, H6, H7, H8, H9: STAND-OFF, SparkFun-Hardware:STAND-OFF
- added LOGO13, LOGO16: SFE_LOGO_NAME_FLAME.3_INCH, SparkFun-Aesthetics:SFE_LOGO_NAME_FLAME_.3
- added LOGO14, LOGO17: OSHW-LOGOM, SparkFun-Aesthetics:OSHW-LOGO-M
- added LOGO15, LOGO18: REVISION, SparkFun-Aesthetics:REVISION
- added Q1, Q2, Q3, Q4, Q5, Q6: 600mA/40V, SparkFun-DiscreteSemi:SOT23-3
- added U$1, U$112, U$149, U$186, U$4, U$75: (no value), buzzard_labels (14):2#7#9V21
- added U$10, U$120, U$157, U$194, U$46, U$83: (no value), buzzard_labels (16):MISO5
- added U$100, U$137, U$174, U$211, U$27, U$63: (no value), buzzard_labels (16):P1411
- added U$101, U$138, U$175, U$212, U$28, U$64: (no value), buzzard_labels (16):P1510
- added U$102, U$139, U$176, U$213, U$29, U$65: (no value), buzzard_labels (16):P1617
- added U$103, U$140, U$177, U$214, U$30, U$66: (no value), buzzard_labels (16):SCK1
- added U$104, U$141, U$178, U$215, U$31, U$67: (no value), buzzard_labels (16):SCL2
- added U$105, U$142, U$179, U$216, U$32, U$68: (no value), buzzard_labels (16):SDA3
- added U$106, U$143, U$180, U$217, U$33, U$69: (no value), buzzard_labels (16):SPI6
- added U$107, U$111, U$144, U$148, U$181, U$185, U$218, U$222, U$34, U$39, U$70, U$74: (no value), buzzard_labels (16):VIN20
- added U$108, U$145, U$182, U$219, U$35, U$71: (no value), buzzard_labels (16):VOUT31
- added U$109, U$123, U$13, U$146, U$160, U$183, U$197, U$220, U$36, U$49, U$72, U$86: (no value), buzzard_labels (16):OFF29
- added U$11, U$121, U$158, U$195, U$47, U$84: (no value), buzzard_labels (16):MOSI4
- added U$110, U$124, U$14, U$147, U$161, U$184, U$198, U$221, U$37, U$50, U$73, U$87: (no value), buzzard_labels (16):ON30
- added U$113, U$150, U$187, U$2, U$38, U$76: (no value), buzzard_labels (14):3#3V25
- added U$114, U$151, U$188, U$3, U$40, U$77: (no value), buzzard_labels (14):5#0V23
- added U$115, U$152, U$189, U$41, U$5, U$78: (no value), buzzard_labels (14):GATOR#BIT26
- added U$116, U$153, U$190, U$42, U$6, U$79: (no value), buzzard_labels (16):GATOR#BIT32
- added U$117, U$118, U$154, U$155, U$191, U$192, U$43, U$44, U$7, U$8, U$80, U$81: (no value), buzzard_labels (16):GND22
- added U$119, U$156, U$193, U$45, U$82, U$9: (no value), buzzard_labels (16):I2C7
- added U$12, U$122, U$159, U$196, U$48, U$85: (no value), buzzard_labels (16):MUSIC28
- added U$125, U$126, U$15, U$16, U$162, U$163, U$199, U$200, U$51, U$52, U$88, U$89: (no value), buzzard_labels (16):OUT24
- added U$127, U$164, U$17, U$201, U$53, U$90: (no value), buzzard_labels (16):P5#A18
- added U$128, U$165, U$18, U$202, U$54, U$91: (no value), buzzard_labels (16):P11#B19
- added U$129, U$166, U$19, U$203, U$55, U$92: (no value), buzzard_labels (16):P013
- added U$130, U$167, U$20, U$204, U$56, U$93: (no value), buzzard_labels (16):P114
- added U$131, U$168, U$205, U$21, U$57, U$94: (no value), buzzard_labels (16):P130
- added U$132, U$169, U$206, U$22, U$58, U$95: (no value), buzzard_labels (16):P199
- added U$133, U$170, U$207, U$23, U$59, U$96: (no value), buzzard_labels (16):P208
- added U$134, U$171, U$208, U$24, U$60, U$97: (no value), buzzard_labels (16):P215
- added U$135, U$172, U$209, U$25, U$61, U$98: (no value), buzzard_labels (16):P816
- added U$136, U$173, U$210, U$26, U$62, U$99: (no value), buzzard_labels (16):P1227
- D10, D12, D13, D15, D17, D19, D25, D26, D27, D28, D44, D8, D86, D87, D88: value 3.8V -> 3.6V; device PDZVTR36BCT:SOD-128 -> SparkFun-DiscreteSemi:SOD-323
- D14, D16, D36, D37, D51: value WS2812B -> 1A/23V/620mV; device SparkFun-LED:WS2812B -> SparkFun-DiscreteSemi:SOD-323
- D18: value WS2812B -> 120mA/40V/370mV; device SparkFun-LED:WS2812B -> SparkFun-DiscreteSemi:SOD-523
- D22, D23, D24, D39, D40, D41, D42, D43, D58, D59, D60: value 3.8V -> WS2812B; device PDZVTR36BCT:SOD-128 -> SparkFun-LED:WS2812B
- D29, D45: value 1A/23V/620mV -> 3.6V
- D30, D31, D46, D47, D48, D63, D64: value RED -> 3.6V; device SparkFun-LED:LED-0603 -> SparkFun-DiscreteSemi:SOD-323
- D32, D94: value RED -> 1A/23V/620mV; device SparkFun-LED:LED-0603 -> SparkFun-DiscreteSemi:SOD-323
- D33, D34, D35, D52, D53: value WS2812B -> RED; device SparkFun-LED:WS2812B -> SparkFun-LED:LED-0603
- D38, D57, D76: value 3.8V -> 120mA/40V/370mV; device PDZVTR36BCT:SOD-128 -> SparkFun-DiscreteSemi:SOD-523
- D49, D50, D65, D66, D67, D68, D69, D82, D83, D84, D85: value WS2812B -> 3.6V; device SparkFun-LED:WS2812B -> SparkFun-DiscreteSemi:SOD-323
- D54, D71, D72, D73, D90, D91, D92: value 3.8V -> RED; device PDZVTR36BCT:SOD-128 -> SparkFun-LED:LED-0603
- D55, D56, D70, D74, D75, D89: value 3.8V -> 1A/23V/620mV; device PDZVTR36BCT:SOD-128 -> SparkFun-DiscreteSemi:SOD-323
- D61, D77: value 1A/23V/620mV -> WS2812B; device SparkFun-DiscreteSemi:SOD-323 -> SparkFun-LED:WS2812B
- D62, D78, D79, D80, D96: value RED -> WS2812B; device SparkFun-LED:LED-0603 -> SparkFun-LED:WS2812B
- D95: value RED -> 120mA/40V/370mV; device SparkFun-LED:LED-0603 -> SparkFun-DiscreteSemi:SOD-523
- J108, J36, J54, J72, J90: value (none) -> POWER_JACKPTH_LOCK; device SparkFun-Connectors:JST-2-SMD -> SparkFun-Connectors:POWER_JACK_PTH_LOCK
- J19: value GATOR -> POWER_JACKPTH_LOCK; device TAB:GATOR -> SparkFun-Connectors:POWER_JACK_PTH_LOCK
- J5: value (none) -> GATOR; device SparkFun-Connectors:JST-2-SMD -> TAB:GATOR
- L1, L2, L3, L4, L5, L6: value 1.5UH -> 1.5uH
- LOGO10, LOGO4: value OSHW-LOGOM -> SFE_LOGO_NAME_FLAME.3_INCH; device SparkFun-Aesthetics:OSHW-LOGO-M -> SparkFun-Aesthetics:SFE_LOGO_NAME_FLAME_.3
- LOGO11, LOGO5: value SFE_LOGO_NAME_FLAME.3_INCH -> OSHW-LOGOM; device SparkFun-Aesthetics:SFE_LOGO_NAME_FLAME_.3 -> SparkFun-Aesthetics:OSHW-LOGO-M
- LOGO12, LOGO6: value OSHW-LOGOM -> REVISION; device SparkFun-Aesthetics:OSHW-LOGO-M -> SparkFun-Aesthetics:REVISION
- LOGO3, LOGO9: value SFE_LOGO_NAME_FLAME.3_INCH -> REVISION; device SparkFun-Aesthetics:SFE_LOGO_NAME_FLAME_.3 -> SparkFun-Aesthetics:REVISION
- R10, R14, R16, R18, R20, R25, R35, R37, R56, R58, R6, R60, R71, R73, R75, R77, R79, R94, R96: value 910 -> 100
- R100: value 910 -> 523k
- R101, R26, R47, R80: value 604 -> 100k
- R102, R48: value 910 -> 390
- R103, R49: value 604 -> 240
- R104, R106, R33, R50, R52: value 910 -> 1k
- R105, R32, R34, R51, R70: value 604 -> 1k
- R107, R38, R41, R61: value 100k -> 100
- R108: value 10.2K -> 10k
- R11, R13, R15, R17, R19, R24, R53, R55, R57, R59, R7, R74, R76, R78, R9, R93, R95, R97: value 604 -> 100
- R27, R81: value 910 -> 10.2K
- R28, R82: value 604 -> 523k
- R29, R83, R98: value 910 -> 100k
- R30: value 604 -> 390
- R31: value 910 -> 240
- R36, R72: value 604 -> 10k
- R39: value 10.2K -> 100
- R40: value 523k -> 100
- R42: value 390k -> 100
- R43, R89: value 240 -> 100
- R44: value 1k -> 100k
- R45: value 1k -> 10.2K
- R46: value 1k -> 523k
- R5: value 390k -> 390
- R54, R8: value 910 -> 10k
- R62: value 10.2K -> 100k
- R63: value 523k -> 10.2K
- R64: value 100k -> 523k
- R65: value 390k -> 100k
- R66: value 240 -> 390
- R67: value 1k -> 240
- R84: value 100k -> 390
- R85: value 10.2K -> 240
- R86: value 523k -> 1k
- R87: value 100k -> 1k
- R88: value 390k -> 1k
- R90: value 1k -> 10k
- R91, R92: value 1k -> 100
- R99: value 604 -> 10.2K
- moved E$1 364.4 mm to (6.86, 142.3)
- moved LOGO12 311.5 mm to (35.1, 59.7)
- moved R59 284.6 mm to (36.8, 87.1)
- moved D57 284.2 mm to (311.4, 40.6), turned to 180 degrees
- moved D51 275.9 mm to (324.9, 16.5), turned to 270 degrees
- moved R60 274.3 mm to (47.0, 87.0)
- moved D55 271.3 mm to (322.3, 16.5)
- moved D50 266.3 mm to (307.1, 20.3), turned to 180 degrees
- moved R58 264.2 mm to (26.7, 87.1)
- moved D54 260.7 mm to (327.3, 38.9), turned to 90 degrees
- moved R61 259.6 mm to (77.6, 87.0), turned to 0 degrees
- moved R68 256.0 mm to (81.3, 108.2), turned to 90 degrees
- moved R63 255.1 mm to (83.7, 99.7), turned to 180 degrees
- moved D53 250.5 mm to (327.3, 56.7), turned to 90 degrees
- moved R69 249.0 mm to (97.8, 133.2)
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Connections:
- removed net N$1 (its old number): LS2.+, S5.3
- removed net N$102: D96.C, R138.2
- removed net N$42 (its old number): R62.2, U10.P$1, U10.P$14
- removed net N$44 (its old number): R63.1, R64.2, U10.P$5
- removed net N$48: D45.C, S11.1
- removed net N$59 (its old number): R85.2, U14.P$1, U14.P$14
- removed net N$62 (its old number): R84.1, U14.P$2
- removed net N$66: D62.C, R90.2
- removed net N$78 (its old number): R109.1, R110.2, U18.P$5
- removed net N$80 (its old number): R111.2, R112.1, U19.1
- removed net N$84: D79.C, R114.2
- removed net N$95 (its old number): R132.1, R133.2, U22.P$5
- removed net N$96 (its old number): R130.1, U22.P$2
- removed net PP0: D12.P$1, R11.2, R14.2
- removed net PP1: D15.P$1, R15.2, R16.2
- removed net PP10: D23.P$1, R26.2, R27.2
- removed net PP11: D10.P$1, R10.2, R9.2
- removed net PP12: D22.P$1, R24.2, R25.2
- removed net PP13: D40.P$1, R51.2, R52.2
- removed net PP14: D41.P$1, R53.2, R54.2
- removed net PP15: D42.P$1, R55.2, R56.2
- removed net PP16: D13.P$1, R13.2, R6.2
- removed net PP17: D43.P$1, R57.2, R58.2
- removed net PP18: D44.P$1, R59.2, R60.2
- removed net PP19: D39.P$1, R49.2, R50.2
- removed net PP2: D17.P$1, R17.2, R18.2
- removed net PP20: D38.P$1, R47.2, R48.2
- removed net PP21: D56.P$1, R74.2, R75.2
- removed net PP22: D57.P$1, R76.2, R77.2
- removed net PP23: D58.P$1, R78.2, R79.2
- removed net PP24: D59.P$1, R80.2, R81.2
- removed net PP25: D60.P$1, R82.2, R83.2
- removed net PP26: D55.P$1, R72.2, R73.2
- removed net PP27: D54.P$1, R70.2, R71.2
- removed net PP28: D72.P$1, R97.2, R98.2
- removed net PP29: D73.P$1, R100.2, R99.2
- removed net PP3: D24.P$1, R28.2, R29.2
- removed net PP30: D74.P$1, R101.2, R102.2
- removed net PP31: D75.P$1, R103.2, R104.2
- removed net PP32: D76.P$1, R105.2, R106.2
- removed net PP33: D71.P$1, R95.2, R96.2
- removed net PP34: D70.P$1, R93.2, R94.2
- removed net PP35: D88.P$1, R120.2, R121.2
- removed net PP36: D89.P$1, R122.2, R123.2
- removed net PP37: D90.P$1, R124.2, R125.2
- removed net PP38: D91.P$1, R126.2, R127.2
- removed net PP39: D92.P$1, R128.2, R129.2
- removed net PP4: D25.P$1, R30.2, R31.2
- removed net PP40: D87.P$1, R118.2, R119.2
- removed net PP41: D86.P$1, R116.2, R117.2
- removed net PP5: D19.P$1, R19.2, R20.2
- removed net PP6: D26.P$1, R32.2, R33.2
- removed net PP7: D27.P$1, R34.2, R35.2
- removed net PP8: D8.P$1, R7.2, R8.2
- removed net PP9: D28.P$1, R36.2, R37.2
- removed net VSUPPLY: S2.2, S4.3
- removed net VSUPPLY1: S7.2, S8.3
- removed net VSUPPLY2: S11.2, S12.3
- removed net VSUPPLY3: S15.2, S16.3
- removed net VSUPPLY4: S19.2, S20.3
- removed net VSUPPLY5: S23.2, S24.3
- new net N$103: D109.C, R104.2
- new net N$104: D110.C, R105.2
- new net N$105: D111.C, R106.2
- new net N$106: R107.2, S11.3
- new net N$107: Q6.1, R107.1
- new net N$108: LS6.-, Q6.3, R108.2
- new net N$21: R27.2, U6.P$1, U6.P$14
- new net N$40: D42.2, D43.4
- new net N$43: R45.2, U10.P$1, U10.P$14
- new net N$47: R48.2, R49.1, U11.1
- new net N$57: D60.2, D61.4
- new net N$58: D61.2, D62.4
- new net N$64: R62.1, U14.P$2
- new net N$74: D78.2, D79.4
- new net N$75: D79.2, D80.4
- new net N$81: R82.1, R83.2, U18.P$5
- new net N$91: D96.2, D97.4
- new net N$92: D97.2, D98.4
- new net N$94: D100.4, D99.2
- net 3.3V: now also D18.A, LS1.+, R8.1; no longer F1.2
- net 3.3V1: now also D38.A, LS2.+, R31.2, R36.1, S4.2; no longer F2.2, R43.2, S6.2
- net 3.3V2: now also D57.A, LS3.+, R49.2, R54.1, S6.2; no longer F3.2, R66.2, S10.2
- net 3.3V3: now also D76.A, LS4.+, R67.2, R72.1, S8.2; no longer F4.2, R89.2, S14.2
- net 3.3V4: now also D95.A, LS5.+, R85.2, R90.1, S10.2; no longer F5.2, R112.2, S18.2
- net 3.3V5: now also D114.A, LS6.+, R103.2, R108.1, S12.2; no longer F6.2, R135.2, S22.2
- net 5V1: now also D22.1, D23.1, D24.1, R26.2, R28.2, S4.5; no longer D14.1, D16.1, D18.1, R38.2, R40.2, S6.5
- net 5V2: now also D39.1, D40.1, D41.1, D42.1, D43.1, R44.2, R46.2, S6.5; no longer D33.1, D34.1, D35.1, D36.1, D37.1, R61.2, R63.2, S10.5
- net 5V3: now also D58.1, D59.1, D60.1, D61.1, D62.1, R62.2, R64.2, S8.5; no longer D49.1, D50.1, D51.1, D52.1, D53.1, R84.2, R86.2, S14.5
- net 5V4: now also D77.1, D78.1, D79.1, D80.1, D81.1, R80.2, R82.2, S10.5; no longer D65.1, D66.1, D67.1, D68.1, D69.1, R107.2, R109.2, S18.5
- net 5V5: now also D100.1, D96.1, D97.1, D98.1, D99.1, R100.2, R98.2, S12.5; no longer D81.1, D82.1, D83.1, D84.1, D85.1, R130.2, R132.2, S22.5
- net GND: now also D10.A, D12.A, D13.A, D15.A, D17.A, D19.A, D8.A, J19.GND, J19.GNDBREAK, Q1.2; no longer D10.P$2, D12.P$2, D13.P$2, D15.P$2, D17.P$2, D19.P$2, D8.P$2, J5.1, LS1.-
- net GND1: now also D22.3, D23.3, D24.3, D25.A, D26.A, D27.A, D28.A, D29.A, D30.A, D31.A, J36.GND, J36.GNDBREAK, Q2.2, R29.1, R30.1, R32.1, R33.1, R34.1; no longer D14.3, D16.3, D18.3, D22.P$2, D23.P$2, D24.P$2, D25.P$2, D26.P$2, D27.P$2, D28.P$2, J36.1, LS2.-, R41.1, R42.1, R44.1, R45.1, R46.1
- net GND2: now also D39.3, D40.3, D41.3, D42.3, D43.3, D44.A, D45.A, D46.A, D47.A, D48.A, D49.A, D50.A, J54.GND, J54.GNDBREAK, Q3.2, R47.1, R48.1, R50.1, R51.1, R52.1; no longer D33.3, D34.3, D35.3, D36.3, D37.3, D38.P$2, D39.P$2, D40.P$2, D41.P$2, D42.P$2, D43.P$2, D44.P$2, J54.1, LS3.-, R64.1, R65.1, R67.1, R68.1, R69.1
- net GND3: now also D58.3, D59.3, D60.3, D61.3, D62.3, D63.A, D64.A, D65.A, D66.A, D67.A, D68.A, D69.A, J72.GND, J72.GNDBREAK, Q4.2, R65.1, R66.1, R68.1, R69.1, R70.1; no longer D49.3, D50.3, D51.3, D52.3, D53.3, D54.P$2, D55.P$2, D56.P$2, D57.P$2, D58.P$2, D59.P$2, D60.P$2, J72.1, LS4.-, R87.1, R88.1, R90.1, R91.1, R92.1
- net GND4: now also D77.3, D78.3, D79.3, D80.3, D81.3, D82.A, D83.A, D84.A, D85.A, D86.A, D87.A, D88.A, J90.GND, J90.GNDBREAK, Q5.2, R83.1, R84.1, R86.1, R87.1, R88.1; no longer D65.3, D66.3, D67.3, D68.3, D69.3, D70.P$2, D71.P$2, D72.P$2, D73.P$2, D74.P$2, D75.P$2, D76.P$2, J90.1, LS5.-, R110.1, R111.1, R113.1, R114.1, R115.1
- net GND5: now also D100.3, D101.A, D102.A, D103.A, D104.A, D105.A, D106.A, D107.A, D96.3, D97.3, D98.3, D99.3, J108.GND, J108.GNDBREAK, Q6.2, R101.1, R102.1, R104.1, R105.1, R106.1; no longer D81.3, D82.3, D83.3, D84.3, D85.3, D86.P$2, D87.P$2, D88.P$2, D89.P$2, D90.P$2, D91.P$2, D92.P$2, J108.1, LS6.-, R133.1, R134.1, R136.1, R137.1, R138.1
- net MBIN: now also D16.A, D18.C; no longer F1.1, S4.1
- net MBIN1: now also D37.A, D38.C; no longer F2.1, S8.1
- net MBIN2: now also D56.A, D57.C; no longer F3.1, S12.1
- net MBIN3: now also D75.A, D76.C; no longer F4.1, S16.1
- net MBIN4: now also D94.A, D95.C; no longer F5.1, S20.1
- net MBIN5: now also D113.A, D114.C; no longer F6.1, S24.1
- net N$10: now also D21.2, D22.4; no longer D14.2, D16.4
- net N$100: now also R98.1, U22.P$2; no longer D94.C, R136.2
- net N$101: now also R102.2, R103.1, U23.1; no longer D95.C, R137.2
- net N$15: now also D22.2, D23.4; no longer D16.2, D18.4
- net N$17: now also D23.2, D24.4; no longer D18.2, D20.4
- net N$20: now also R6.2, S3.3; no longer D6.C, S2.1
- net N$25: now also Q1.1, R6.1; no longer R39.2, U6.P$1, U6.P$14
- net N$27: now also R28.1, R29.2; no longer R40.1, R41.2
- net N$28: now also R26.1; no longer R38.1
- net N$29: now also R30.2, R31.1; no longer R42.2, R43.1
- net N$3: now also LS1.-, Q1.3, R8.2; no longer LS1.+, S3.3
- net N$31: now also D33.C, R32.2; no longer D29.C, S7.1
- net N$32: now also D34.C, R33.2; no longer D30.C, R44.2
- net N$33: now also D35.C, R34.2; no longer D31.C, R45.2
- net N$34: now also R35.2, S2.3; no longer D32.C, R46.2
- net N$35: now also Q2.1, R35.1; no longer LS3.+, S9.3
- net N$36: now also LS2.-, Q2.3, R36.2; no longer D33.2, D34.4
- net N$37: now also D39.2, D40.4; no longer D34.2, D35.4
- net N$38: now also D40.2, D41.4; no longer D35.2, D36.4
- net N$39: now also D41.2, D42.4; no longer D36.2, D37.4
- net N$45: now also R46.1, R47.2, U10.P$5; no longer R61.1, U10.P$2
- net N$46: now also R44.1, U10.P$2; no longer R65.2, R66.1, U11.1
- net N$49: now also D52.C, R50.2; no longer D46.C, R67.2
- net N$50: now also D53.C, R51.2; no longer D47.C, R68.2
- net N$51: now also D54.C, R52.2; no longer D48.C, R69.2
- net N$52: now also R53.2, S5.3; no longer LS4.+, S13.3
- net N$53: now also Q3.1, R53.1; no longer D49.2, D50.4
- net N$54: now also LS3.-, Q3.3, R54.2; no longer D50.2, D51.4
- net N$55: now also D58.2, D59.4; no longer D51.2, D52.4
- net N$56: now also D59.2, D60.4; no longer D52.2, D53.4
- net N$61: now also R63.2, U14.P$1, U14.P$14; no longer R86.1, R87.2, U14.P$5
- net N$63: now also R64.1, R65.2, U14.P$5; no longer R88.2, R89.1, U15.1
- net N$65: now also R66.2, R67.1, U15.1; no longer D61.C, S15.1
- net N$67: now also D71.C, R68.2; no longer D63.C, R91.2
- net N$68: now also D72.C, R69.2; no longer D64.C, R92.2
- net N$69: now also D73.C, R70.2; no longer LS5.+, S17.3
- net N$70: now also R71.2, S7.3; no longer D65.2, D66.4
- net N$71: now also Q4.1, R71.1; no longer D66.2, D67.4
- net N$72: now also LS4.-, Q4.3, R72.2; no longer D67.2, D68.4
- net N$73: now also D77.2, D78.4; no longer D68.2, D69.4
- net N$76: now also D80.2, D81.4; no longer R108.2, U18.P$1, U18.P$14
- net N$79: now also R81.2, U18.P$1, U18.P$14; no longer R107.1, U18.P$2
- net N$82: now also R80.1, U18.P$2; no longer D77.C, S19.1
- net N$83: now also R84.2, R85.1, U19.1; no longer D78.C, R113.2
- net N$85: now also D90.C, R86.2; no longer D80.C, R115.2
- net N$86: now also D91.C, R87.2; no longer LS6.+, S21.3
- net N$87: now also D92.C, R88.2; no longer D81.2, D82.4
- net N$88: now also R89.2, S9.3; no longer D82.2, D83.4
- net N$89: now also Q5.1, R89.1; no longer D83.2, D84.4
- net N$90: now also LS5.-, Q5.3, R90.2; no longer D84.2, D85.4
- net N$93: now also D98.2, D99.4; no longer R131.2, U22.P$1, U22.P$14
- net N$97: now also R99.2, U22.P$1, U22.P$14; no longer R134.2, R135.1, U23.1
- net N$99: now also R100.1, R101.2, U22.P$5; no longer D93.C, S23.1
- net P0+1: now also R18.1; no longer R30.1
- net P0+2: now also R40.1; no longer R53.1
- net P0+3: now also R58.1; no longer R76.1
- net P0+4: now also R76.1; no longer R99.1
- net P0+5: now also R94.1; no longer R122.1
- net P1: now also D15.C, R15.2; no longer R16.1
- net P1+1: now also R20.1; no longer R32.1
- net P1+2: now also R41.1; no longer R55.1
- net P1+3: now also R59.1; no longer R78.1
- net P1+4: now also R77.1; no longer R101.1
- net P1+5: now also R95.1; no longer R124.1
- net P10: now also D20.4; no longer D14.4
- net P11: now also D10.C, R9.2; no longer R10.1
- net P11+1: now also R16.1; no longer R28.1
- net P11+2: now also R39.1; no longer R51.1
- net P11+3: now also R57.1; no longer R74.1
- net P11+4: now also R75.1; no longer R97.1
- net P11+5: now also R93.1; no longer R120.1
- net P16: now also D13.C, R13.2; no longer R6.1
- net P16+1: now also R10.1; no longer R24.1
- net P16+2: now also R37.1; no longer R47.1
- net P16+3: now also R55.1; no longer R70.1
- net P16+4: now also R73.1; no longer R93.1
- net P16+5: now also R91.1; no longer R116.1
- net P17: now also D30.C, R24.2; no longer R35.1
- net P2: now also D17.C, R17.2; no longer R18.1
- net P2+1: now also R24.1; no longer R34.1
- net P2+2: now also R42.1; no longer R57.1
- net P2+3: now also R60.1; no longer R80.1
- net P2+4: now also R78.1; no longer R103.1
- net P2+5: now also R96.1; no longer R126.1
- net P23: now also D25.C, R10.2; no longer R25.1
- net P26: now also D46.C, R39.2; no longer R52.1
- net P27: now also D50.C, R43.2; no longer R60.1
- net P28: now also S5.2; no longer S9.2
- net P29: now also D48.C, R41.2; no longer R56.1
- net P3: now also D27.C, R16.2; no longer R29.1
- net P30: now also D45.C, R38.2; no longer R50.1
- net P31: now also D39.4; no longer D33.4
- net P32: now also D49.C, R42.2; no longer R58.1
- net P36: now also D44.C, R37.2; no longer R48.1
- net P39: now also D65.C, R57.2; no longer R75.1
- net P4: now also D31.C, R25.2; no longer R37.1
- net P40: now also D69.C, R61.2; no longer R83.1
- net P41: now also S7.2; no longer S13.2
- net P42: now also D67.C, R59.2; no longer R79.1
- net P43: now also D64.C, R56.2; no longer R73.1
- net P44: now also D58.4; no longer D49.4
- net P45: now also D68.C, R60.2; no longer R81.1
- net P49: now also D63.C, R55.2; no longer R71.1
- net P5: now also D19.C, R19.2; no longer R20.1
- net P5+1: now also R25.1; no longer R36.1
- net P5+2: now also R43.1; no longer R59.1
- net P5+3: now also R61.1; no longer R82.1
- net P5+4: now also R79.1; no longer R105.1
- net P5+5: now also R97.1; no longer R128.1
- net P52: now also D84.C, R75.2; no longer R98.1
- net P53: now also D88.C, R79.2; no longer R106.1
- net P54: now also S9.2; no longer S17.2
- net P55: now also D86.C, R77.2; no longer R102.1
- net P56: now also D83.C, R74.2; no longer R96.1
- net P57: now also D77.4; no longer D65.4
- net P58: now also D87.C, R78.2; no longer R104.1
- net P6: now also S2.2; no longer S5.2
- net P62: now also D82.C, R73.2; no longer R94.1
- net P65: now also D103.C, R93.2; no longer R121.1
- net P66: now also D107.C, R97.2; no longer R129.1
- net P67: now also S11.2; no longer S21.2
- net P68: now also D105.C, R95.2; no longer R125.1
- net P69: now also D102.C, R92.2; no longer R119.1
- net P7: now also D29.C, R20.2; no longer R33.1
- net P70: now also D96.4; no longer D81.4
- net P71: now also D106.C, R96.2; no longer R127.1
- net P75: now also D101.C, R91.2; no longer R117.1
- net P8: now also D8.C, R7.2; no longer R8.1
- net P8+1: now also R14.1; no longer R26.1
- net P8+2: now also R38.1; no longer R49.1
- net P8+3: now also R56.1; no longer R72.1
- net P8+4: now also R74.1; no longer R95.1
- net P8+5: now also R92.1; no longer R118.1
- net P9: now also D26.C, R14.2; no longer R27.1
- net PD: now also D12.C, R11.2; no longer R14.1
- net PD1: now also D28.C, R18.2, S2.1; no longer R31.1, S5.1
- net PD2: now also D47.C, R40.2, S5.1; no longer R54.1, S9.1
- net PD3: now also D66.C, R58.2, S7.1; no longer R77.1, S13.1
- net PD4: now also D85.C, R76.2, S9.1; no longer R100.1, S17.1
- net PD5: now also D104.C, R94.2, S11.1; no longer R123.1, S21.1
- net VIN: now also D14.C, D16.C, D6.C; no longer S4.2
- net VIN1: now also D32.C, D33.A, D36.C, D37.C, R27.1; no longer D30.A, R39.1, S8.2
- net VIN2: now also D51.C, D52.A, D55.C, D56.C, R45.1; no longer D46.A, R62.1, S12.2
- net VIN3: now also D70.C, D71.A, D74.C, D75.C, R63.1; no longer D62.A, R85.1, S16.2
- net VIN4: now also D89.C, D90.A, D93.C, D94.C, R81.1; no longer D78.A, R108.1, S20.2
- net VIN5: now also D108.C, D109.A, D112.C, D113.C, R99.1; no longer D94.A, R131.1, S24.2
- net VIN_TAB1: now also D32.A; no longer D29.A
- net VIN_TAB2: now also D51.A; no longer D45.A
- net VIN_TAB3: now also D70.A; no longer D61.A
- net VIN_TAB4: now also D89.A; no longer D77.A
- net VIN_TAB5: now also D108.A; no longer D93.A
- net VOUT3.1: now also D34.A, J5.P$1, J5.P$2, S4.3; no longer D31.A, J19.P$1, J19.P$2, S6.3
- net VOUT3.2: now also D53.A, S6.3; no longer D47.A, S10.3
- net VOUT3.4: now also D72.A, S8.3; no longer D63.A, S14.3
- net VOUT3.5: now also D91.A, S10.3; no longer D79.A, S18.3
- net VOUT3.6: now also D110.A, S12.3; no longer D95.A, S22.3
- net VOUT5.1: now also D35.A, S4.6; no longer D32.A, S6.6
- net VOUT5.2: now also D54.A, S6.6; no longer D48.A, S10.6
- net VOUT5.3: now also D73.A, S8.6; no longer D64.A, S14.6
- net VOUT5.4: now also D92.A, S10.6; no longer D80.A, S18.6
- net VOUT5.5: now also D111.A, S12.6; no longer D96.A, S22.6
- net V_BATT: now also D14.A, J19.PWR; no longer J5.2, S2.3
- net V_BATT1: now also D36.A, J36.PWR; no longer J36.2, S7.3
- net V_BATT2: now also D55.A, J54.PWR; no longer J54.2, S11.3
- net V_BATT3: now also D74.A, J72.PWR; no longer J72.2, S15.3
- net V_BATT4: now also D93.A, J90.PWR; no longer J90.2, S19.3
- net V_BATT5: now also D112.A, J108.PWR; no longer J108.2, S23.3
Routing:
- net VSUPPLY: track 46.3 -> 0.00 mm, vias 2 -> 0
- net VSUPPLY3: track 46.3 -> 0.00 mm, vias 2 -> 0
- net VSUPPLY4: track 46.3 -> 0.00 mm, vias 2 -> 0
- net VSUPPLY1: track 46.3 -> 0.00 mm, vias 2 -> 0
- net VSUPPLY5: track 46.3 -> 0.00 mm, vias 2 -> 0
- net VSUPPLY2: track 46.3 -> 0.00 mm, vias 2 -> 0
- net 3.3V: track 143.6 -> 170.2 mm, vias 0 -> 2
- net 3.3V1: track 143.6 -> 170.2 mm, vias 0 -> 2
- net 3.3V3: track 143.6 -> 170.2 mm, vias 0 -> 2
- net 3.3V4: track 143.6 -> 170.2 mm, vias 0 -> 2
- net 3.3V2: track 143.6 -> 170.2 mm, vias 0 -> 2
- net 3.3V5: track 143.6 -> 170.2 mm, vias 0 -> 2
- net N$108: track 0.00 -> 23.2 mm
- net GND5: track 68.5 -> 45.9 mm, vias 52 -> 50
- net GND2: track 68.5 -> 45.9 mm, vias 52 -> 50
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- added copper zone on layer 16, net N$102
- added copper zone on layer 16, net N$48
- added copper zone on layer 16, net N$66
- added copper zone on layer 16, net N$84
- removed copper zone on layer 16, net N$47
- removed copper zone on layer 16, net N$64
- removed copper zone on layer 16, net N$81
- removed copper zone on layer 16, net N$98 (its old number)
Other:
- board size 357.8 x 155 mm -> 364 x 160.3 mm
- board text added: "Andy England"
- board text added: "Mary West"
- board text added: "v-score"
- board text added: "v20"
- board text removed: "2.7-9V"
- board text removed: "5.0V"
- board text removed: "BATT"
- board text removed: "GND"
- board text removed: "I2C"
- board text removed: "MISO"
- board text removed: "MOSI"
- board text removed: "MUSIC"
- board text removed: "OFF"
- board text removed: "ON"
- board text removed: "OUT"
- board text removed: "P0"
- board text removed: "P1"
- board text removed: "P11/B"
- board text removed: "P12"
- board text removed: "P13"
- board text removed: "P14"
- board text removed: "P15"
- board text removed: "P16"
- board text removed: "P19"
- board text removed: "P2"
- board text removed: "P20"
- board text removed: "P5/A"
- board text removed: "P8"
- board text removed: "POWER"
- board text removed: "PWR In"
- board text removed: "Power in"
- board text removed: "SCK"
- board text removed: "SCL"
- board text removed: "SDA"
- board text removed: "SPI"
- board text removed: "TAB"
- board text removed: "USB"
- board text removed: "VIN"
- board text removed: "VOUT"
- board text removed: "gator:bit"
- board text removed: "route out"
- board text removed: "v10"
